Commit message: Updated URDF Files to newer versions.

File: reach5mini_simulation/urdf/reach5mini.gazebo.xacro (robot description, xacro)
@@ -1,68 +1,70 @@
 <?xml version="1.0"?>
 <robot name="reach5mini_sim" xmlns:xacro="http://ros.org/wiki/xacro">
-  <transmission name="trans_joint5">
-      <type>transmission_interface/SimpleTransmission</type>
-      <joint name="joint5">
-          <hardwareInterface>hardware_interface/PositionJointInterface</hardwareInterface>
-      </joint>
-      <actuator name="joint5_motor">
-          <hardwareInterface>hardware_interface/PositionJointInterface</hardwareInterface>
-          <mechanicalReduction>1</mechanicalReduction>
-      </actuator>
-  </transmission>
-  <transmission name="trans_joint4">
-      <type>transmission_interface/SimpleTransmission</type>
-      <joint name="joint4">
-          <hardwareInterface>hardware_interface/PositionJointInterface</hardwareInterface>
-      </joint>
-      <actuator name="joint4_motor">
-          <hardwareInterface>hardware_interface/PositionJointInterface</hardwareInterface>
-          <mechanicalReduction>1</mechanicalReduction>
-      </actuator>
-  </transmission>
-  <transmission name="trans_joint3">
-      <type>transmission_interface/SimpleTransmission</type>
-      <joint name="joint3">
-          <hardwareInterface>hardware_interface/PositionJointInterface</hardwareInterface>
-      </joint>
-      <actuator name="joint3_motor">
-          <hardwareInterface>hardware_interface/PositionJointInterface</hardwareInterface>
-          <mechanicalReduction>1</mechanicalReduction>
-      </actuator>
-  </transmission>
-  <transmission name="trans_joint2">
-      <type>transmission_interface/SimpleTransmission</type>
-      <joint name="joint2">
-          <hardwareInterface>hardware_interface/PositionJointInterface</hardwareInterface>
-      </joint>
-      <actuator name="joint2_motor">
-          <hardwareInterface>hardware_interface/PositionJointInterface</hardwareInterface>
-          <mechanicalReduction>1</mechanicalReduction>
-      </actuator>
-  </transmission>
-  <transmission name="trans_joint1_2">
-      <type>transmission_interface/SimpleTransmission</type>
-      <joint name="joint1_2">
-          <hardwareInterface>hardware_interface/PositionJointInterface</hardwareInterface>
-      </joint>
-      <actuator name="joint1_2_motor">
-          <hardwareInterface>hardware_interface/PositionJointtInterface</hardwareInterface>
-          <mechanicalReduction>1</mechanicalReduction>
-      </actuator>
-  </transmission>
-  <transmission name="trans_joint1_1">
-      <type>transmission_interface/SimpleTransmission</type>
-      <joint name="joint1_1">
-          <hardwareInterface>hardware_interface/PositionJointInterface</hardwareInterface>
-      </joint>
-      <actuator name="joint1_1_motor">
-          <hardwareInterface>hardware_interface/PositionJointInterface</hardwareInterface>
-          <mechanicalReduction>1</mechanicalReduction>
-      </actuator>
-  </transmission>
-  <gazebo>
-      <plugin name="gazebo_ros_control" filename="libgazebo_ros_control.so">
-          <robotNamespace>/</robotNamespace>
-      </plugin>
-  </gazebo>
+  <xacro:macro name="reach5mini_gazebo" params="name:=reach5mini">
+    <transmission name="${name}_trans_joint5">
+        <type>transmission_interface/SimpleTransmission</type>
+        <joint name="${name}_joint5">
+            <hardwareInterface>hardware_interface/PositionJointInterface</hardwareInterface>
+        </joint>
+        <actuator name="${name}_joint5_motor">
+            <hardwareInterface>hardware_interface/PositionJointInterface</hardwareInterface>
+            <mechanicalReduction>1</mechanicalReduction>
+        </actuator>
+    </transmission>
+    <transmission name="${name}_trans_joint4">
+        <type>transmission_interface/SimpleTransmission</type>
+        <joint name="${name}_joint4">
+            <hardwareInterface>hardware_interface/PositionJointInterface</hardwareInterface>
+        </joint>
+        <actuator name="${name}_joint4_motor">
+            <hardwareInterface>hardware_interface/PositionJointInterface</hardwareInterface>
+            <mechanicalReduction>1</mechanicalReduction>
+        </actuator>
+    </transmission>
+    <transmission name="${name}_trans_joint3">
+        <type>transmission_interface/SimpleTransmission</type>
+        <joint name="${name}_joint3">
+            <hardwareInterface>hardware_interface/PositionJointInterface</hardwareInterface>
+        </joint>
+        <actuator name="${name}_joint3_motor">
+            <hardwareInterface>hardware_interface/PositionJointInterface</hardwareInterface>
+            <mechanicalReduction>1</mechanicalReduction>
+        </actuator>
+    </transmission>
+    <transmission name="${name}_trans_joint2">
+        <type>transmission_interface/SimpleTransmission</type>
+        <joint name="${name}_joint2">
+            <hardwareInterface>hardware_interface/PositionJointInterface</hardwareInterface>
+        </joint>
+        <actuator name="${name}_joint2_motor">
+            <hardwareInterface>hardware_interface/PositionJointInterface</hardwareInterface>
+            <mechanicalReduction>1</mechanicalReduction>
+        </actuator>
+    </transmission>
+    <transmission name="${name}_trans_joint1_2">
+        <type>transmission_interface/SimpleTransmission</type>
+        <joint name="${name}_joint1_2">
+            <hardwareInterface>hardware_interface/PositionJointInterface</hardwareInterface>
+        </joint>
+        <actuator name="${name}_joint1_2_motor">
+            <hardwareInterface>hardware_interface/PositionJointtInterface</hardwareInterface>
+            <mechanicalReduction>1</mechanicalReduction>
+        </actuator>
+    </transmission>
+    <transmission name="${name}_trans_joint1_1">
+        <type>transmission_interface/SimpleTransmission</type>
+        <joint name="${name}_joint1_1">
+            <hardwareInterface>hardware_interface/PositionJointInterface</hardwareInterface>
+        </joint>
+        <actuator name="${name}_joint1_1_motor">
+            <hardwareInterface>hardware_interface/PositionJointInterface</hardwareInterface>
+            <mechanicalReduction>1</mechanicalReduction>
+        </actuator>
+    </transmission>
+    <gazebo>
+        <plugin name="gazebo_ros_control" filename="libgazebo_ros_control.so">
+            <robotNamespace></robotNamespace>
+        </plugin>
+    </gazebo>
+  </xacro:macro>
 </robot>

File: reach5mini_simulation/urdf/reach5mini.urdf.xacro (robot description, xacro)
@@ -6,203 +6,211 @@
     <xacro:include filename="$(find reach5mini_simulation)/urdf/reach5mini.gazebo.xacro"/>
   </xacro:if>
-  <xacro:if value="$(arg fixed)">
-    <link name="world"/>
-    <joint name="fixed" type="fixed">
-      <parent link="world"/>
-      <child link="base_link"/>
+  <xacro:macro name="reach5mini" params="parent *origin name:=reach5mini">
+    <reach5mini_gazebo name="${name}"/>
+    <!-- camera body, with origin at bottom screw mount -->
+    <joint name="${name}_joint" type="fixed">
+      <xacro:insert_block name="origin" />
+      <parent link="${parent}"/>
+      <child link="${name}_base_link" />
     </joint>
-  </xacro:if>
-    <material name="black">
-        <color rgba="0 0 0 1" />
-    </material>
-    <link name="base_link">
-        <visual>
-            <geometry>
-                <mesh filename="package://reach5mini_description/meshes/Base.stl" />
-            </geometry>
-            <origin rpy="0 0 0" xyz="0 0 0" />
-            <material name="black" />
-        </visual>
-        <collision>
-            <geometry>
-                <cylinder length="0.150" radius="0.020" />
-            </geometry>
-            <origin rpy="0 1.57075 0" xyz="-0.075 0 0" />
-        </collision>
-        <inertial>
-            <mass value="0.341" />
-            <origin xyz="-0.075 -0.006 -0.003" />
-            <inertia ixx="0.000099" ixy="0.000139" ixz="0.000115" iyy="0.002920" iyz="0.000003" izz="0.002934" />
-        </inertial>
-    </link>
-    <link name="shoulder_link">
-        <visual>
-            <geometry>
-                <mesh filename="package://reach5mini_description/meshes/ShoulderJoint.stl" />
-            </geometry>
-            <material name="black" />
-            <origin rpy="0 0 -1.57075" xyz="0 0 0" />
-        </visual>
-        <collision>
-            <geometry>
-                <cylinder length="0.066" radius="0.020" />
-            </geometry>
-            <origin rpy="0 0 0" xyz="0 0 0.010" />
-        </collision>
-        <inertial>
-            <mass value="0.194" />
-            <origin xyz="0.005 -0.001 0.016" />
-            <inertia ixx="0.000189" ixy="0.000005" ixz="0.000054" iyy="0.000213" iyz="0.000003" izz="0.000067" />
-        </inertial>
-    </link>
-    <link name="upper_arm_link">
-        <visual>
-            <geometry>
-                <mesh filename="package://reach5mini_description/meshes/UpperArm.stl" />
-            </geometry>
-            <origin rpy="0 -1.57075 -0.2655555" xyz="0 0 -0.075" />
-            <material name="black" />
-        </visual>
-        <collision>
-            <geometry>
-                <cylinder length="0.145" radius="0.020" />
-            </geometry>
-            <origin rpy="0 1.57075 -0.27075" xyz="0.075 0 0" />
-        </collision>
-        <collision>
-            <geometry>
-                <cylinder length="0.040" radius="0.020" />
-            </geometry>
-            <origin rpy="0 0 0" xyz="0 0 0" />
-        </collision>
-        <inertial>
-            <mass value="0.429" />
-            <origin xyz="0.073 0.0 0.0" />
-            <inertia ixx="0.000087" ixy="-0.000076" ixz="-0.000010" iyy="0.003190" iyz="0.000000" izz="0.003213" />
-        </inertial>
-    </link>
-    <link name="forearm_link">
-        <visual>
-            <geometry>
-                <mesh filename="package://reach5mini_description/meshes/ForearmJoint.stl" />
-            </geometry>
-            <origin rpy="0 0 0" xyz="0 0 0" />
-            <material name="black" />
-        </visual>
-        <collision>
-            <geometry>
-                <cylinder length="0.040" radius="0.020" />
-            </geometry>
-            <origin rpy="0 0 0" xyz="0 0 0" />
-        </collision>
-        <inertial>
-            <mass value="0.115" />
-            <origin xyz="0.017 -0.026 -0.002" />
-            <inertia ixx="0.000120" ixy="-0.000061" ixz="-0.000001" iyy="0.000062" iyz="0.000000" izz="0.000156" />
-        </inertial>
-    </link>
-    <link name="wrist_link">
-        <visual>
-            <geometry>
-                <mesh filename="package://reach5mini_description/meshes/Wrist.stl" />
-            </geometry>
-            <origin rpy="0 0 0" xyz="0 0 0" />
-            <material name="black" />
-        </visual>
-        <collision>
-            <geometry>
-                <cylinder length="0.140" radius="0.020" />
-            </geometry>
-            <origin rpy="0 0 0" xyz="0 0 -0.070" />
-        </collision>
-        <inertial>
-            <mass value="0.333" />
-            <origin xyz="0.0 0.003 -0.098" />
-            <inertia ixx="0.003709" ixy="-0.000002" ixz="-0.000004" iyy="0.003734" iyz="0.000000" izz="0.000079" />
-        </inertial>
-    </link>
-    <link name="jaw1">
-        <visual>
-            <geometry>
-                <mesh filename="package://reach5mini_description/meshes/Jaw1.stl" />
-            </geometry>
-            <origin rpy="0 0 0" xyz="0 0 0" />
-            <material name="black" />
-        </visual>
-        <collision>
-            <geometry>
-                <box size="0.03 0.09 0.01" />
-            </geometry>
-            <origin rpy="0 0 0" xyz="-0.01 -0.045 0" />
-        </collision>
-        <!-- TODO: GET APPROPOATE MASSES - John Sumskas -->
-        <inertial>
-            <mass value="0.194" />
-            <origin xyz="0.005 -0.001 0.016" />
-            <inertia ixx="0.000189" ixy="0.000005" ixz="0.000054" iyy="0.000213" iyz="0.000003" izz="0.000067" />
-        </inertial>
-    </link>
-    <link name="jaw2">
-        <visual>
-            <geometry>
-                <mesh filename="package://reach5mini_description/meshes/Jaw2.stl" />
-            </geometry>
-            <origin rpy="0 0 0" xyz="0 0 0" />
-            <material name="black" />
-        </visual>
-        <collision>
-            <geometry>
-                <box size="0.03 0.09 0.01" />
-            </geometry>
-            <origin rpy="0 0 0" xyz="0.01 -0.045 0" />
-        </collision>
-        <!-- TODO: GET APPROPOATE MASSES - John Sumskas -->
-        <inertial>
-            <mass value="0.194" />
-            <origin xyz="0.005 -0.001 0.016" />
-            <inertia ixx="0.000189" ixy="0.000005" ixz="0.000054" iyy="0.000213" iyz="0.000003" izz="0.000067" />
-        </inertial>
-    </link>
-    <joint name="joint5" type="revolute">
-        <parent link="base_link" />
-        <child link="shoulder_link" />
-        <origin xyz="0 0 0" rpy="0 0 3.141592" />
-        <axis xyz="0 0 1" />
-        <limit effort="9.0" lower="0.0" upper="6.2" velocity="0.5" />
-    </joint>
-    <joint name="joint4" type="revolute">
-        <parent link="shoulder_link" />
-        <child link="upper_arm_link" />
-        <origin xyz="0.020 0 0.046" rpy="1.57075 1.3 0" />
-        <axis xyz="0 0 1" />
-        <limit effort="9.0" lower="0.0" upper="3.5" velocity="0.5" />
-    </joint>
-    <joint name="joint3" type="revolute">
-        <parent link="upper_arm_link" />
-        <child link="forearm_link" />
-        <origin xyz="0.15 0 0" rpy="3.1415 0 1.3" />
-        <axis xyz="0 0 1" />
-        <limit effort="9.0" lower="0.0" upper="3.5" velocity="0.5" />
-    </joint>
-    <joint name="joint2" type="revolute">
-        <parent link="forearm_link" />
-        <child link="wrist_link" />
-        <origin xyz="0.020 0 0" rpy="-1.57075 0 0" />
-        <axis xyz="0 0 1" />
-        <limit effort="5.0" lower="0.0" upper="6.0" velocity="1.0" />
-    </joint>
-    <joint name="joint1_2" type="revolute">
-        <parent link="wrist_link" />
-        <child link="jaw1" />
-        <origin xyz="0.015 0 -0.140" rpy="1.57075 0 0" />
-        <axis xyz="0 0 1" />
-        <limit effort="5.0" lower="0.0" upper="0.5" velocity="0.5" />
-    </joint>
-    <joint name="joint1_1" type="revolute">
-        <parent link="wrist_link" />
-        <child link="jaw2" />
-        <origin xyz="-0.015 0 -0.140" rpy="1.57075 0 0" />
-        <axis xyz="0 0 -1" />
-        <limit effort="5.0" lower="0.0" upper="0.5" velocity="0.5" />
-    </joint>
+      <material name="black">
+          <color rgba="0 0 0 1" />
+      </material>
+      <link name="${name}_base_link">
+          <visual>
+              <geometry>
+                  <mesh filename="package://reach5mini_simulation/meshes/Base.stl" />
+              </geometry>
+              <origin rpy="0 0 0" xyz="0 0 0" />
+              <material name="black" />
+          </visual>
+          <collision>
+              <geometry>
+                  <cylinder length="0.150" radius="0.020" />
+              </geometry>
+              <origin rpy="0 1.57075 0" xyz="-0.075 0 0" />
+          </collision>
+          <inertial>
+              <mass value="0.341" />
+              <origin xyz="-0.075 -0.006 -0.003" />
+              <inertia ixx="0.000099" ixy="0.000139" ixz="0.000115" iyy="0.002920" iyz="0.000003" izz="0.002934" />
+          </inertial>
+      </link>
+      <link name="${name}_shoulder_link">
+          <visual>
+              <geometry>
+                  <mesh filename="package://reach5mini_simulation/meshes/ShoulderJoint.stl" />
+              </geometry>
+              <material name="black" />
+              <origin rpy="0 0 -1.57075" xyz="0 0 0" />
+          </visual>
+          <collision>
+              <geometry>
+                  <cylinder length="0.066" radius="0.020" />
+              </geometry>
+              <origin rpy="0 0 0" xyz="0 0 0.010" />
+          </collision>
+          <inertial>
+              <mass value="0.194" />
+              <origin xyz="0.005 -0.001 0.016" />
+              <inertia ixx="0.000189" ixy="0.000005" ixz="0.000054" iyy="0.000213" iyz="0.000003" izz="0.000067" />
+          </inertial>
+      </link>
+      <link name="${name}_upper_arm_link">
+          <visual>
+              <geometry>
+                  <mesh filename="package://reach5mini_simulation/meshes/UpperArm.stl" />
+              </geometry>
+              <origin rpy="0 -1.57075 -0.2655555" xyz="0 0 -0.075" />
+              <material name="black" />
+          </visual>
+          <collision>
+              <geometry>
+                  <cylinder length="0.145" radius="0.020" />
+              </geometry>
+              <origin rpy="0 1.57075 -0.27075" xyz="0.075 0 0" />
+          </collision>
+          <collision>
+              <geometry>
+                  <cylinder length="0.040" radius="0.020" />
+              </geometry>
+              <origin rpy="0 0 0" xyz="0 0 0" />
+          </collision>
+          <inertial>
+              <mass value="0.429" />
+              <origin xyz="0.073 0.0 0.0" />
+              <inertia ixx="0.000087" ixy="-0.000076" ixz="-0.000010" iyy="0.003190" iyz="0.000000" izz="0.003213" />
+          </inertial>
+      </link>
+      <link name="${name}_forearm_link">
+          <visual>
+              <geometry>
+                  <mesh filename="package://reach5mini_simulation/meshes/ForearmJoint.stl" />
+              </geometry>
+              <origin rpy="0 0 0" xyz="0 0 0" />
+              <material name="black" />
+          </visual>
+          <collision>
+              <geometry>
+                  <cylinder length="0.040" radius="0.020" />
+              </geometry>
+              <origin rpy="0 0 0" xyz="0 0 0" />
+          </collision>
+          <inertial>
+              <mass value="0.115" />
+              <origin xyz="0.017 -0.026 -0.002" />
+              <inertia ixx="0.000120" ixy="-0.000061" ixz="-0.000001" iyy="0.000062" iyz="0.000000" izz="0.000156" />
+          </inertial>
+      </link>
+      <link name="${name}_wrist_link">
+          <visual>
+              <geometry>
+                  <mesh filename="package://reach5mini_simulation/meshes/Wrist.stl" />
+              </geometry>
+              <origin rpy="0 0 0" xyz="0 0 0" />
+              <material name="black" />
+          </visual>
+          <collision>
+              <geometry>
+                  <cylinder length="0.140" radius="0.020" />
+              </geometry>
+              <origin rpy="0 0 0" xyz="0 0 -0.070" />
+          </collision>
+          <inertial>
+              <mass value="0.333" />
+              <origin xyz="0.0 0.003 -0.098" />
+              <inertia ixx="0.003709" ixy="-0.000002" ixz="-0.000004" iyy="0.003734" iyz="0.000000" izz="0.000079" />
+          </inertial>
+      </link>
+      <link name="${name}_jaw1">
+          <visual>
+              <geometry>
+                  <mesh filename="package://reach5mini_simulation/meshes/Jaw1.stl" />
+              </geometry>
+              <origin rpy="0 0 0" xyz="0 0 0" />
+              <material name="black" />
+          </visual>
+          <collision>
+              <geometry>
+                  <box size="0.03 0.09 0.01" />
+              </geometry>
+              <origin rpy="0 0 0" xyz="-0.01 -0.045 0" />
+          </collision>
+          <!-- TODO: GET APPROPOATE MASSES - John Sumskas -->
+          <inertial>
+              <mass value="0.194" />
+              <origin xyz="0.005 -0.001 0.016" />
+              <inertia ixx="0.000189" ixy="0.000005" ixz="0.000054" iyy="0.000213" iyz="0.000003" izz="0.000067" />
+          </inertial>
+      </link>
+      <link name="${name}_jaw2">
+          <visual>
+              <geometry>
+                  <mesh filename="package://reach5mini_simulation/meshes/Jaw2.stl" />
+              </geometry>
+              <origin rpy="0 0 0" xyz="0 0 0" />
+              <material name="black" />
+          </visual>
+          <collision>
+              <geometry>
+                  <box size="0.03 0.09 0.01" />
+              </geometry>
+              <origin rpy="0 0 0" xyz="0.01 -0.045 0" />
+          </collision>
+          <!-- TODO: GET APPROPOATE MASSES - John Sumskas -->
+          <inertial>
+              <mass value="0.194" />
+              <origin xyz="0.005 -0.001 0.016" />
+              <inertia ixx="0.000189" ixy="0.000005" ixz="0.000054" iyy="0.000213" iyz="0.000003" izz="0.000067" />
+          </inertial>
+      </link>
+      <joint name="${name}_joint1_1" type="revolute">
+          <parent link="${name}_wrist_link" />
+          <child link="${name}_jaw2" />
+          <origin xyz="-0.015 0 -0.140" rpy="1.57075 0 0" />
+          <axis xyz="0 0 -1" />
+          <limit effort="5.0" lower="0.0" upper="0.5" velocity="0.5" />
+      </joint>
+      <joint name="${name}_joint1_2" type="revolute">
+          <parent link="${name}_wrist_link" />
+          <child link="${name}_jaw1" />
+          <origin xyz="0.015 0 -0.140" rpy="1.57075 0 0" />
+          <axis xyz="0 0 1" />
+          <limit effort="5.0" lower="0.0" upper="0.5" velocity="0.5" />
+      </joint>
+      <joint name="${name}_joint2" type="revolute">
+          <parent link="${name}_forearm_link" />
+          <child link="${name}_wrist_link" />
+          <origin xyz="0.020 0 0" rpy="-1.57075 -0.5 0" />
+          <axis xyz="0 0 1" />
+          <limit effort="5.0" lower="0.0" upper="6.0" velocity="1.0" />
+      </joint>
+      <joint name="${name}_joint3" type="revolute">
+          <parent link="${name}_upper_arm_link" />
+          <child link="${name}_forearm_link" />
+          <origin xyz="0.15 0 0" rpy="3.1415 0 1.3" />
+          <axis xyz="0 0 1" />
+          <limit effort="9.0" lower="0.0" upper="3.5" velocity="0.5" />
+      </joint>
+      <joint name="${name}_joint4" type="revolute">
+          <parent link="${name}_shoulder_link" />
+          <child link="${name}_upper_arm_link" />
+          <origin xyz="0.020 0 0.046" rpy="1.57075 1.3 0" />
+          <axis xyz="0 0 1" />
+          <limit effort="9.0" lower="0.0" upper="3.5" velocity="0.5" />
+      </joint>
+      <joint name="${name}_joint5" type="revolute">
+          <parent link="${name}_base_link" />
+          <child link="${name}_shoulder_link" />
+          <origin xyz="0 0 0" rpy="0 0 3.141592" />
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